Commit message: add ur5 arm urdf

File: mr_pkg/urdf/ur5.urdf (robot description, URDF)
Before this commit: robot ur5, 5 links, 4 joints
Links:
- removed link link1
- removed link link2
- removed link link3
- added link ee_link
- added link forearm_link; visual mesh filename=package://mr_pkg/meshes/ur5/visual/forearm.dae
- added link shoulder_link; visual mesh filename=package://mr_pkg/meshes/ur5/visual/shoulder.dae
- added link upper_arm_link; visual mesh filename=package://mr_pkg/meshes/ur5/visual/upperarm.dae
- added link wrist_1_link; visual mesh filename=package://mr_pkg/meshes/ur5/visual/wrist1.dae
- added link wrist_2_link; visual mesh filename=package://mr_pkg/meshes/ur5/visual/wrist2.dae
- added link wrist_3_link; visual mesh filename=package://mr_pkg/meshes/ur5/visual/wrist3.dae
- link base_link: mass 4.0 -> None; geometry visual mesh filename=package://mr_pkg/meshes/ur5/visual/base.dae
Joints:
- removed joint joint1
- removed joint joint2
- removed joint joint3
- added joint ee_joint: type fixed, parent wrist_3_link, child ee_link, origin xyz=0.0 0.082 0.0 rpy=0.0 0.0 0.0
- added joint elbow_joint: type continuous, parent upper_arm_link, child forearm_link, origin xyz=0.425 0 0 rpy=0.0 0.0 0.0, axis 0.0 1.0 0.0
- added joint shoulder_1_joint: type continuous, parent base_link, child shoulder_link, origin xyz=0.0 0.0 0.089 rpy=0.0 0.0 0.0, axis 0.0 0.0 1.0
- added joint shoulder_2_joint: type continuous, parent shoulder_link, child upper_arm_link, origin xyz=0.0 0.109 0.0 rpy=0.0 0.0 0.0, axis 0.0 1.0 0.0
- added joint wrist_1_joint: type continuous, parent forearm_link, child wrist_1_link, origin xyz=0.392 0 0 rpy=0.0 0.0 0.0, axis 0.0 1.0 0.0
- added joint wrist_2_joint: type continuous, parent wrist_1_link, child wrist_2_link, origin xyz=0.0 0.0 0.0 rpy=0.0 0.0 0.0, axis 0.0 0.0 -1.0
- added joint wrist_3_joint: type continuous, parent wrist_2_link, child wrist_3_link, origin xyz=0 0 -0.095 rpy=0.0 0.0 0.0, axis 0.0 1.0 0.0

Commit message: finsih exe8

File: mr_pkg/urdf/ur5.urdf (robot description, URDF)
Before this commit: robot ur5, 9 links, 8 joints
Joints:
- joint ee_joint: origin xyz=0.0 0.082 0.0 rpy=0.0 0.0 0.0 -> xyz=0.0 0.082 0.0 rpy=-1.570796325 0.0 0.0
- joint elbow_joint: origin xyz=0.425 0 0 rpy=0.0 0.0 0.0 -> xyz=0.0 -0.1197 0.425 rpy=0.0 0.0 0.0
- joint shoulder_1_joint: origin xyz=0.0 0.0 0.089 rpy=0.0 0.0 0.0 -> xyz=0.0 0.0 0.089159 rpy=0.0 0.0 0.0
- joint shoulder_2_joint: origin xyz=0.0 0.109 0.0 rpy=0.0 0.0 0.0 -> xyz=0.0 0.13585 0.0 rpy=0.0 1.570796325 0.0
- joint wrist_1_joint: origin xyz=0.392 0 0 rpy=0.0 0.0 0.0 -> xyz=0.0 0 0.39225 rpy=0.0 1.570796325 0.0
- joint wrist_2_joint: axis 0.0 0.0 -1.0 -> 0.0 0.0 1.0; origin xyz=0.0 0.0 0.0 rpy=0.0 0.0 0.0 -> xyz=0.0 0.093 0.0 rpy=0.0 0.0 0.0
- joint wrist_3_joint: origin xyz=0 0 -0.095 rpy=0.0 0.0 0.0 -> xyz=0 0 0.09465 rpy=0.0 0.0 0.0
